File: 006P-5VSupply/006P-5VSupply-TLV1117.brd (EAGLE design)
At the start: 100 x 80 mm, 16 parts, among them IC1 TLV1117-33

Commit message: Update 006P-5VSupply Project
Parts:
- R4: value 100 -> 33
Changed lines of the file:
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@@
 <element name="R3" library="rcl" package="0207/7" value="1k" x="16.51" y="27.94" rot="R180"/>
 <element name="IC1" library="ic-package" package="DIL10" value="TLV1117-33" x="10.16" y="-7.62"/>
-<element name="R4" library="rcl" package="0207/7" value="100" x="5.08" y="-17.78"/>
+<element name="R4" library="rcl" package="0207/7" value="33" x="5.08" y="-17.78"/>
 <element name="S1" library="switch" package="TL3XPO" value="TL36PO" x="7.62" y="-25.4"/>
 </elements>
