File: 006P-5VSupply/006P-5VSupply-TLV1117.sch (EAGLE design)
At the start: 16 parts, among them IC1 TLV1117-33

Commit message: Update 006P-5VSupply Project
Parts:
- R4: value 100 -> 33
Changed lines of the file:
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@@
 <part name="R3" library="rcl" deviceset="R-EU_" device="0207/7" value="1k"/>
 <part name="IC1" library="ic-package" deviceset="DIL10" device="" value="TLV1117-33"/>
-<part name="R4" library="rcl" deviceset="R-EU_" device="0207/7" value="100"/>
+<part name="R4" library="rcl" deviceset="R-EU_" device="0207/7" value="33"/>
 <part name="S1" library="switch" deviceset="TL36PO" device=""/>
 </parts>
