File: 006P-5VSupply/006P-5VSupply.brd (EAGLE design)
At the start: 100 x 80 mm, 14 parts, among them IC1 7805T

Commit message: Update 006P-5VSupply Project
Parts:
- removed C2: 10u, rcl:E2-4
- removed D3: 1N4004, diode:DO41-10
- removed R1: 240, rcl:0207/7
- removed R2: 5k, rcl:RTRIM3339P
- R3: value 1k -> 10k
- moved D1 43.4 mm to (10.2, 12.7)
- moved JP4 32.8 mm to (14.0, 2.54), turned to 180 degrees
- moved C3 32.4 mm to (14.0, 7.62), turned to 180 degrees
- moved C1 25.7 mm to (6.35, 7.62), turned to 0 degrees
- moved C5 23.3 mm to (14.0, 15.2), turned to 180 degrees
- moved R3 21.6 mm to (2.54, 11.4), turned to 270 degrees
- moved C4 21.6 mm to (6.35, 15.2), turned to 0 degrees
- moved IC1 21.6 mm to (10.2, 27.9)
- moved JP2 20.1 mm to (6.35, 2.54), turned to 180 degrees
- moved LED1 15.5 mm to (2.54, 19.1), turned to 90 degrees
Connections:
- removed net N$3: C2.+, D3.A, IC1.2, R1.1, R2.3
- net GND: now also IC1.2; no longer C2.-, R2.1, R2.2
- net N$1: no longer D3.C, R1.2
Routing:
- net N$1: track 63.8 -> 18.3 mm
- net N$3: track 31.0 -> 0.00 mm
- net GND: track 67.1 -> 41.4 mm
- net N$4: track 41.1 -> 21.1 mm
- net N$6: track 7.62 -> 2.54 mm
Changed lines of the file:
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@@
 </autorouter>
 <elements>
-<element name="C1" library="rcl" package="E2-4" value="47u" x="15.24" y="31.75" rot="R270"/>
-<element name="C2" library="rcl" package="E2-4" value="10u" x="35.56" y="21.59" rot="R270"/>
-<element name="C3" library="rcl" package="E2-4" value="47u" x="35.56" y="31.75" rot="R270"/>
-<element name="C4" library="rcl" package="C025-024X044" value="0.1u" x="20.32" y="31.75" rot="R270"/>
-<element name="C5" library="rcl" package="C025-024X044" value="0.1u" x="30.48" y="31.75" rot="R270"/>
-<element name="D1" library="diode" package="DO41-10" value="1N4004" x="25.4" y="53.34"/>
-<element name="D3" library="diode" package="DO41-10" value="1N4004" x="30.48" y="22.86" rot="R270"/>
-<element name="IC1" library="linear" package="TO220H" value="7805T" x="25.4" y="43.18"/>
-<element name="JP2" library="pinhead" package="1X02" value="VIN9V" x="12.7" y="21.59" rot="R90"/>
-<element name="JP4" library="pinhead" package="1X02" value="VOUT5V" x="40.64" y="21.59" rot="R270"/>
-<element name="LED1" library="led" package="LED3MM" value="" x="17.78" y="21.59" rot="R270"/>
-<element name="R1" library="rcl" package="0207/7" value="240" x="36.83" y="17.78"/>
-<element name="R2" library="rcl" package="RTRIM3339P" value="5k" x="25.4" y="22.86" rot="R90"/>
-<element name="R3" library="rcl" package="0207/7" value="1k" x="16.51" y="27.94" rot="R180"/>
+<element name="C1" library="rcl" package="E2-4" value="47u" x="6.35" y="7.62"/>
+<element name="C3" library="rcl" package="E2-4" value="47u" x="13.97" y="7.62" rot="R180"/>
+<element name="C4" library="rcl" package="C025-024X044" value="0.1u" x="6.35" y="15.24"/>
+<element name="C5" library="rcl" package="C025-024X044" value="0.1u" x="13.97" y="15.24" rot="R180"/>
+<element name="D1" library="diode" package="DO41-10" value="1N4004" x="10.16" y="12.7"/>
+<element name="IC1" library="linear" package="TO220H" value="7805T" x="10.16" y="27.94"/>
+<element name="JP2" library="pinhead" package="1X02" value="VIN9V" x="6.35" y="2.54" rot="R180"/>
+<element name="JP4" library="pinhead" package="1X02" value="VOUT5V" x="13.97" y="2.54" rot="R180"/>
+<element name="LED1" library="led" package="LED3MM" value="" x="2.54" y="19.05" rot="R90"/>
+<element name="R3" library="rcl" package="0207/7" value="10k" x="2.54" y="11.43" rot="R270"/>
 </elements>
 <signals>
 <signal name="N$1">
 <contactref element="IC1" pad="3"/>
-<contactref element="D3" pad="C"/>
-<contactref element="R1" pad="2"/>
 <contactref element="C5" pad="1"/>
 <contactref element="C3" pad="+"/>
 <contactref element="D1" pad="A"/>
 <contactref element="JP4" pad="1"/>
-<wire x1="30.48" y1="33.02" x2="27.94" y2="33.02" width="0.4064" layer="16"/>
-<wire x1="30.48" y1="33.02" x2="35.56" y2="33.02" width="0.4064" layer="16"/>
-<wire x1="40.64" y1="22.86" x2="40.64" y2="27.94" width="0.4064" layer="16"/>
-<wire x1="40.64" y1="27.94" x2="40.64" y2="33.02" width="0.4064" layer="16"/>
-<wire x1="40.64" y1="33.02" x2="35.56" y2="33.02" width="0.4064" layer="16"/>
-<wire x1="35.56" y1="33.02" x2="35.56" y2="32.766" width="0.4064" layer="16"/>
-<wire x1="30.48" y1="27.94" x2="40.64" y2="27.94" width="0.4064" layer="16"/>
-<wire x1="40.64" y1="22.86" x2="43.18" y2="22.86" width="0.4064" layer="16"/>
-<wire x1="43.18" y1="22.86" x2="43.18" y2="17.78" width="0.4064" layer="16"/>
-<wire x1="43.18" y1="17.78" x2="40.64" y2="17.78" width="0.4064" layer="16"/>
-<wire x1="30.48" y1="53.34" x2="30.48" y2="33.02" width="0.4064" layer="16"/>
-</signal>
-<signal name="N$3">
-<contactref element="IC1" pad="2"/>
-<contactref element="R1" pad="1"/>
-<contactref element="D3" pad="A"/>
-<contactref element="C2" pad="+"/>
-<contactref element="R2" pad="3"/>
-<wire x1="25.4" y1="33.02" x2="25.4" y2="25.4" width="0.4064" layer="16"/>
-<wire x1="25.4" y1="25.4" x2="35.56" y2="25.4" width="0.4064" layer="16"/>
-<wire x1="35.56" y1="25.4" x2="35.56" y2="22.606" width="0.4064" layer="16"/>
-<wire x1="30.48" y1="17.78" x2="33.02" y2="17.78" width="0.4064" layer="16"/>
-<wire x1="33.02" y1="17.78" x2="33.02" y2="22.86" width="0.4064" layer="1"/>
-<wire x1="33.02" y1="22.86" x2="35.56" y2="22.86" width="0.4064" layer="1"/>
-<wire x1="35.56" y1="22.86" x2="35.56" y2="22.606" width="0.4064" layer="1"/>
+<wire x1="12.7" y1="17.78" x2="15.24" y2="17.78" width="0.4064" layer="16"/>
+<wire x1="15.24" y1="17.78" x2="15.24" y2="15.24" width="0.4064" layer="16"/>
+<wire x1="15.24" y1="15.24" x2="15.24" y2="12.7" width="0.4064" layer="16"/>
+<wire x1="15.24" y1="12.7" x2="14.986" y2="12.7" width="0.4064" layer="16"/>
+<wire x1="14.986" y1="12.7" x2="14.986" y2="7.62" width="0.4064" layer="16"/>
+<wire x1="14.986" y1="7.62" x2="15.24" y2="7.62" width="0.4064" layer="16"/>
+<wire x1="15.24" y1="7.62" x2="15.24" y2="2.54" width="0.4064" layer="16"/>
 </signal>
 <signal name="N$4">
@@
 <contactref element="JP2" pad="2"/>
 <contactref element="R3" pad="2"/>
-<wire x1="12.7" y1="22.86" x2="12.7" y2="27.94" width="0.4064" layer="16"/>
-<wire x1="12.7" y1="27.94" x2="12.7" y2="33.02" width="0.4064" layer="16"/>
-<wire x1="12.7" y1="33.02" x2="15.24" y2="33.02" width="0.4064" layer="16"/>
-<wire x1="15.24" y1="33.02" x2="15.24" y2="32.766" width="0.4064" layer="16"/>
-<wire x1="15.24" y1="32.766" x2="20.32" y2="32.766" width="0.4064" layer="16"/>
-<wire x1="20.32" y1="32.766" x2="20.32" y2="33.02" width="0.4064" layer="16"/>
-<wire x1="20.32" y1="33.02" x2="22.86" y2="33.02" width="0.4064" layer="16"/>
-<wire x1="20.32" y1="53.34" x2="20.32" y2="33.02" width="0.4064" layer="16"/>
+<wire x1="7.62" y1="17.78" x2="5.08" y2="17.78" width="0.4064" layer="16"/>
+<wire x1="5.08" y1="17.78" x2="5.08" y2="15.24" width="0.4064" layer="16"/>
+<wire x1="5.08" y1="15.24" x2="5.08" y2="12.7" width="0.4064" layer="16"/>
+<wire x1="5.08" y1="12.7" x2="5.334" y2="12.7" width="0.4064" layer="16"/>
+<wire x1="5.334" y1="12.7" x2="5.334" y2="7.62" width="0.4064" layer="16"/>
+<wire x1="5.334" y1="7.62" x2="5.08" y2="7.62" width="0.4064" layer="16"/>
+<wire x1="5.08" y1="7.62" x2="5.08" y2="2.54" width="0.4064" layer="16"/>
+<wire x1="2.54" y1="7.62" x2="5.334" y2="7.62" width="0.4064" layer="16"/>
 </signal>
 <signal name="GND">
 <contactref element="C1" pad="-"/>
 <contactref element="C4" pad="2"/>
-<contactref element="C2" pad="-"/>
 <contactref element="C3" pad="-"/>
 <contactref element="C5" pad="2"/>
@@
 <contactref element="JP4" pad="2"/>
 <contactref element="LED1" pad="K"/>
-<contactref element="R2" pad="1"/>
-<contactref element="R2" pad="2"/>
-<wire x1="12.7" y1="20.32" x2="17.78" y2="20.32" width="0.4064" layer="16"/>
-<wire x1="25.4" y1="20.32" x2="27.94" y2="20.32" width="0.4064" layer="16"/>
-<wire x1="27.94" y1="20.574" x2="27.94" y2="22.86" width="0.4064" layer="16"/>
-<wire x1="35.56" y1="20.574" x2="27.94" y2="20.574" width="0.4064" layer="16"/>
-<wire x1="27.94" y1="20.574" x2="27.94" y2="20.32" width="0.4064" layer="16"/>
-<wire x1="40.64" y1="20.574" x2="40.64" y2="20.32" width="0.4064" layer="16"/>
-<wire x1="15.24" y1="30.734" x2="20.32" y2="30.734" width="0.4064" layer="16"/>
-<wire x1="20.32" y1="30.734" x2="20.32" y2="30.48" width="0.4064" layer="16"/>
-<wire x1="40.64" y1="20.32" x2="35.56" y2="20.32" width="0.4064" layer="16"/>
-<wire x1="35.56" y1="20.32" x2="35.56" y2="20.574" width="0.4064" layer="16"/>
-<wire x1="30.48" y1="30.48" x2="35.56" y2="30.48" width="0.4064" layer="16"/>
-<wire x1="35.56" y1="30.48" x2="35.56" y2="30.734" width="0.4064" layer="16"/>
-<wire x1="27.94" y1="22.86" x2="22.86" y2="22.86" width="0.4064" layer="16"/>
-<wire x1="22.86" y1="22.86" x2="22.86" y2="30.48" width="0.4064" layer="16"/>
-<wire x1="22.86" y1="30.48" x2="20.32" y2="30.48" width="0.4064" layer="16"/>
-<wire x1="17.78" y1="20.32" x2="25.4" y2="20.32" width="0.4064" layer="16"/>
-<wire x1="30.48" y1="30.48" x2="20.32" y2="30.48" width="0.4064" layer="1"/>
+<contactref element="IC1" pad="2"/>
+<wire x1="7.62" y1="15.24" x2="10.16" y2="15.24" width="0.4064" layer="16"/>
+<wire x1="10.16" y1="15.24" x2="12.7" y2="15.24" width="0.4064" layer="16"/>
+<wire x1="10.16" y1="17.78" x2="10.16" y2="15.24" width="0.4064" layer="16"/>
+<wire x1="7.366" y1="7.62" x2="7.62" y2="7.62" width="0.4064" layer="16"/>
+<wire x1="7.62" y1="7.62" x2="7.62" y2="2.54" width="0.4064" layer="16"/>
+<wire x1="7.62" y1="2.54" x2="12.7" y2="2.54" width="0.4064" layer="16"/>
+<wire x1="12.7" y1="2.54" x2="12.954" y2="2.54" width="0.4064" layer="16"/>
+<wire x1="12.954" y1="2.54" x2="12.954" y2="7.62" width="0.4064" layer="16"/>
+<wire x1="12.954" y1="7.62" x2="12.7" y2="7.62" width="0.4064" layer="16"/>
+<wire x1="12.7" y1="7.62" x2="12.7" y2="15.24" width="0.4064" layer="16"/>
+<wire x1="2.54" y1="20.32" x2="10.16" y2="20.32" width="0.4064" layer="16"/>
+<wire x1="10.16" y1="20.32" x2="10.16" y2="17.78" width="0.4064" layer="16"/>
 </signal>
 <signal name="N$6">
 <contactref element="R3" pad="1"/>
 <contactref element="LED1" pad="A"/>
-<wire x1="20.32" y1="27.94" x2="20.32" y2="22.86" width="0.4064" layer="16"/>
-<wire x1="20.32" y1="22.86" x2="17.78" y2="22.86" width="0.4064" layer="16"/>
+<wire x1="2.54" y1="15.24" x2="2.54" y2="17.78" width="0.4064" layer="16"/>
 </signal>
 </signals>
