File: SQR_FG/SQR_FG.sch (EAGLE design)
At the start: 24 parts, among them IC1 MEGA328P, IC2 NJM7032, Q1 16MHz, SW1 EC12E_SW

Commit message: Update SQR_FG.sch, SQR_FG.brd
Parts:
- removed R10: 10k, pot:3RP/1610N
- removed R2: 10k/B, pot:3RP/1610N
- removed SW1: EC12E_SW, switch-alps:EC12E_SW
- added C10, C11, C14: 47uF, rcl:CPOL-EUTT2D5L
- added C12, C13, C8, C9: 0.1uF, rcl:C-EU025-024X044
- added D1: 1N4007, diode:1N4004
- added IC3: 7805T, linear:7805T
- added IC4: TLV1117-33, ic-package:DIL10
- added JP3: Duty, pinhead:PINHD-1X3
- added JP4: Encoder, pinhead:PINHD-1X4
- added JP5: Level, pinhead:PINHD-1X3
- added JP6: 9V, pinhead:PINHD-1X2
- C6: value (none) -> 22pF
- R3: value 33k -> 10k
- T1, T2: value (none) -> 2SK4017
Connections:
- net +3V3: now also C13.1, IC4.5
- net +5V: now also C10.+, C11.+, C12.1, C14.+, C8.1, C9.1, IC3.VI, IC3.VO, IC4.3, JP3.1, JP6.1; no longer R2.A
- net GND: now also C10.-, C11.-, C12.2, C13.2, C14.-, C8.2, C9.2, IC3.GND, IC4.1, JP3.3, JP4.4, JP6.2; no longer R2.E, SW1G$1.C, SW1G$2.1
- net N$15: now also JP5.2
- net N$6: now also JP5.3; no longer R10.A
- net N$8: now also JP5.1; no longer R10.E
- net N$9: now also JP3.2; no longer R2.S
- net RE_A: now also JP4.1; no longer SW1G$1.B
- net RE_B: now also JP4.2; no longer SW1G$1.A
- net RE_SW: now also JP4.3; no longer SW1G$2.2
Other:
- note removed: "Rotary Encoder"
- moved on the sheet: R3
